File: hardware/hackrf-one/mcu.kicad_sch (KiCad schematic)
At the start: 132 parts, among them J1 USB-MICRO-B, P1 1V8, P20 GPIO, P22 I2S, P23 DBGEN, P24 TRST, P25 LPC_ISP, P26 LPC_JTAG, P28 SD, P29 CPLD_JTAG, P3 GND, P30 BANK2_AUX, P5 LEDS, P68 SPIFI_CS, P69 VREGMODE, P70 EN_1V8, P71 ID, P72 GP_CLKIN, P73 P1_2, P74 P1_1, P75 GP_CLKIN, P76 GP_CLKIN, P77 GP_CLKIN, P78 GP_CLKIN, P79 GP_CLKIN, P8 VCC, P80 SHIELD, P81 SPIFI_SIO2, P82 SPIFI_SIO3, Q5 MOSFET_P, SW1 DFU, SW2 RESET, U15 USB6B1, U20 W25Q80, U21 TPS62410, U23 LPC4320FBD144, U24 GSG-XC2C64A-7VQG100C, X2 MCU_XTAL, X3 RTC_XTAL

Commit message: Attempts to resolve wierd legacy ERC errors
Connections:
- net +1.8V: no longer C125.1, C126.1, C127.1, L10.2, P1.2 (PM), R47.1
- new net REG_OUT2: C125.1, C126.1, C127.1, L10.2, P1.2 (PM), R47.1
Other:
- moved on the sheet: C127, J1, P1, P80
